File: IO_block.kicad_sch (KiCad schematic)
At the start: 20 parts, among them J5 Conn_01x04, Q4 AO3401A, Q4 BC847, Q5 BC847

Commit message: before scripts
Parts:
- removed R19 (x2): DNP/1210, Resistor_SMD:R_1210_3225Metric_Pad1.30x2.65mm_HandSolder, symbol Device:R_Small
- added C10: 100n, Capacitor_SMD:C_0402_1005Metric, symbol Device:C_Small
- added F1: 1812_2A, Fuse:Fuse_1812_4532Metric, symbol Device:Polyfuse
- added JP6: IN_BYP, Jumper:SolderJumper-2_P1.3mm_Open_TrianglePad1.0x1.5mm, symbol Jumper:SolderJumper_2_Open
- added JP6: OUT_BYP, Jumper:SolderJumper-2_P1.3mm_Open_TrianglePad1.0x1.5mm, symbol Jumper:SolderJumper_2_Open
- added Q5: BC847, Package_TO_SOT_SMD:SOT-23, symbol Transistor_BJT:BC847
- added R19 (x4): 10k, Resistor_SMD:R_0402_1005Metric, symbol Device:R_Small
- added R19: 1k, Resistor_SMD:R_0402_1005Metric, symbol Device:R_Small
- added R19: 330/0.1%, Resistor_SMD:R_0402_1005Metric, symbol Device:R_Small
- added R2: 50mR/1206, Resistor_SMD:R_1206_3216Metric_Pad1.30x1.75mm_HandSolder, symbol Device:R
- added U6: LMV321, Package_TO_SOT_SMD:SOT-23-5, symbol Amplifier_Operational:LMV321
- J5: footprint Connector_Wire:SolderWire-0.127sqmm_1x04_P3.7mm_D0.48mm_OD1mm -> TerminalBlock:TerminalBlock_bornier-4_P5.08mm
Connections:
- net +3.3V: now also C10.1, R19.1, U6.5 (V+)
- net GND: now also C10.2, Q5.2 (E), R19.2, R2.2, U6.2 (V-); no longer J5.4 (Pin_4)
- net IN: now also JP6.2 (B)
- net OUT: now also JP6.2 (B), R19.2; no longer Q5.1 (B)
- net PWR_ENA: now also R19.2; no longer Q4.1 (G), R20.1
- net OUT_BANK: now reaches J5.2 (Pin_2), Q5.3 (C), R19.1
- net OUT_BANK: now also JP6.1 (A)
- net INP_BANK: now reaches D2.2 (A2), J5.3 (Pin_3), R19.1
- net at C10.1, Q4.1 (B), R19.2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: now also JP6.1 (A)
- net at Q4.3 (D): now also F1.1; no longer J5.1 (Pin_1)
- new net: Q5.1 (B), R19.1 (x2)
- new net: Q4.1 (G), Q5.3 (C), R20.1
- new net: R19.1, R19.2, U6.4
- new net: R19.1, R19.2, U6.3 (-)
- new net CURR: R19.1, R19.2
- new net GND_BANK: J5.4 (Pin_4), R2.1, U6.1 (+)
- new net PWR_BANK: F1.2, J5.1 (Pin_1)
Other:
- note added: "Offset for software calibration"
- note added: "YOLO measurement Imax=2A dRload@2A = 100mV target amp = 30 amp = 1+ (Rf / Rg) = 1 + 10k/0.33k = 31.3"
- note added: "reference (link)"
- moved on the sheet: D3, Q4, R19, R20

Commit message: production
Parts:
- C10: LCSC (none) -> C1525
- D3: LCSC (none) -> C3019524
- F1: LCSC (none) -> C20999
- Q4, Q5: LCSC (none) -> C8512
- R19: LCSC (none) -> C25744
- R2: LCSC C601102 -> C25905
- R20: LCSC C25117 -> C912768
- U6: LCSC (none) -> C7972
Changed lines of the file:
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@@
       (effects (font (size 1.27 1.27)) (justify left) hide)
     )
+    (property "LCSC" "C8512" (at 154.7113 61.5863 0)
+      (effects (font (size 1.27 1.27)) hide)
+    )
     (pin "1")
     (pin "2")
@@
     )
     (property "Datasheet" "~" (at 111.76 109.22 0)
+      (effects (font (size 1.27 1.27)) hide)
+    )
+    (property "LCSC" "C25744" (at 109.22 107.95 0)
       (effects (font (size 1.27 1.27)) hide)
     )
@@
       (effects (font (size 1.27 1.27)) hide)
     )
+    (property "LCSC" "C25744" (at 134.62 118.11 0)
+      (effects (font (size 1.27 1.27)) hide)
+    )
     (pin "1")
     (pin "2")
@@
     )
     (property "Datasheet" "~" (at 247.65 57.15 0)
+      (effects (font (size 1.27 1.27)) hide)
+    )
+    (property "LCSC" "C25744" (at 245.11 55.88 0)
       (effects (font (size 1.27 1.27)) hide)
     )
@@
       (effects (font (size 1.27 1.27)) (justify left) hide)
     )
+    (property "LCSC" "C8512" (at 114.0713 88.2563 0)
+      (effects (font (size 1.27 1.27)) hide)
+    )
     (pin "1")
     (pin "2")
@@
       (effects (font (size 1.27 1.27)) hide)
     )
+    (property "LCSC" "C25744" (at 214.63 55.88 0)
+      (effects (font (size 1.27 1.27)) hide)
+    )
     (pin "1")
     (pin "2")
@@
     )
     (property "Datasheet" "~" (at 138.43 62.23 0)
+      (effects (font (size 1.27 1.27)) hide)
+    )
+    (property "LCSC" "C25744" (at 138.43 59.69 0)
       (effects (font (size 1.27 1.27)) hide)
     )
@@
       (effects (font (size 1.27 1.27)) (justify left) hide)
     )
+    (property "LCSC" "C8512" (at 165.227 53.7753 0)
+      (effects (font (size 1.27 1.27)) hide)
+    )
     (pin "1")
     (pin "2")
@@
       (effects (font (size 1.27 1.27)) hide)
     )
+    (property "LCSC" "C25744" (at 214.63 60.96 0)
+      (effects (font (size 1.27 1.27)) hide)
+    )
     (pin "1")
     (pin "2")
@@
       (effects (font (size 1.27 1.27)) hide)
     )
-    (property "LCSC" "C25117" (at 121.92 123.19 0)
+    (property "LCSC" "C912768" (at 121.92 123.19 0)
       (effects (font (size 1.27 1.27)) hide)
     )
@@
       (effects (font (size 1.27 1.27)) hide)
     )
+    (property "LCSC" "C25744" (at 210.82 118.11 0)
+      (effects (font (size 1.27 1.27)) hide)
+    )
     (pin "1")
     (pin "2")
@@
       (effects (font (size 1.27 1.27)) hide)
     )
+    (property "LCSC" "C3019524" (at 229.4128 48.5394 0)
+      (effects (font (size 1.27 1.27)) hide)
+    )
     (pin "1")
     (pin "2")
@@
       (effects (font (size 1.27 1.27)) hide)
     )
+    (property "LCSC" "C25744" (at 114.3 76.2 0)
+      (effects (font (size 1.27 1.27)) hide)
+    )
     (pin "1")
     (pin "2")
@@
       (effects (font (size 1.27 1.27)) hide)
     )
+    (property "LCSC" "C1525" (at 128.4859 122.3616 0)
+      (effects (font (size 1.27 1.27)) hide)
+    )
     (pin "1")
     (pin "2")
@@
       (effects (font (size 1.27 1.27)) hide)
     )
-    (property "LCSC" "C601102" (at 161.29 122.555 0)
+    (property "LCSC" "C25905" (at 161.29 122.555 0)
       (effects (font (size 1.27 1.27)) hide)
     )
@@
       (effects (font (size 1.27 1.27)) hide)
     )
+    (property "LCSC" "C1525" (at 179.2859 108.3916 0)
+      (effects (font (size 1.27 1.27)) hide)
+    )
     (pin "1")
     (pin "2")
@@
       (effects (font (size 1.27 1.27)) hide)
     )
+    (property "LCSC" "C25744" (at 185.42 133.35 0)
+      (effects (font (size 1.27 1.27)) hide)
+    )
     (pin "1")
     (pin "2")
@@
       (effects (font (size 1.27 1.27)) hide)
     )
+    (property "LCSC" "C25744" (at 229.87 55.88 0)
+      (effects (font (size 1.27 1.27)) hide)
+    )
     (pin "1")
     (pin "2")
@@
       (effects (font (size 1.27 1.27)) hide)
     )
+    (property "LCSC" "C25744" (at 170.18 123.19 0)
+      (effects (font (size 1.27 1.27)) hide)
+    )
     (pin "1")
     (pin "2")
@@
       (effects (font (size 1.27 1.27)) hide)
     )
+    (property "LCSC" "C25744" (at 219.71 115.57 0)
+      (effects (font (size 1.27 1.27)) hide)
+    )
     (pin "1")
     (pin "2")
@@
     )
     (property "Datasheet" "~" (at 100.33 88.9 0)
+      (effects (font (size 1.27 1.27)) hide)
+    )
+    (property "LCSC" "C25744" (at 100.33 86.36 0)
       (effects (font (size 1.27 1.27)) hide)
     )
@@
       (effects (font (size 1.27 1.27)) hide)
     )
+    (property "LCSC" "C20999" (at 164.719 81.9063 0)
+      (effects (font (size 1.27 1.27)) hide)
+    )
     (pin "1")
     (pin "2")
@@
       (effects (font (size 1.27 1.27)) (justify left) hide)
     )
+    (property "LCSC" "C8512" (at 109.4487 118.7363 0)
+      (effects (font (size 1.27 1.27)) hide)
+    )
     (pin "1")
     (pin "2")
@@
       (effects (font (size 1.27 1.27)) hide)
     )
+    (property "LCSC" "C7972" (at 201.2818 117.5131 0)
+      (effects (font (size 1.27 1.27)) hide)
+    )
     (pin "2")
     (pin "5")
@@
     )
     (property "Datasheet" "~" (at 247.65 49.53 0)
+      (effects (font (size 1.27 1.27)) hide)
+    )
+    (property "LCSC" "C3019524" (at 244.6528 48.5394 0)
       (effects (font (size 1.27 1.27)) hide)
     )
@@
       (effects (font (size 1.27 1.27)) hide)
     )
-    (property "LCSC" "C25117" (at 152.4 49.53 0)
+    (property "LCSC" "C912768" (at 152.4 49.53 0)
       (effects (font (size 1.27 1.27)) hide)
     )
@@
       (effects (font (size 1.27 1.27)) hide)
     )
+    (property "LCSC" "C3019524" (at 214.1728 48.5394 0)
+      (effects (font (size 1.27 1.27)) hide)
+    )
