File: IO_block.kicad_sch (KiCad schematic)
At the start: 31 parts, among them J5 Conn_01x04, Q4 AO3401A, Q4 BC847, Q5 BC847, U6 LMV321

Commit message: add license, update readme
Parts:
- renumbered C10 to C5, D2 to D3, D3 to D4, D3 to D5, D3 to D6, JP6 to JP11, JP6 to JP7, Q5 to Q15, Q4 to Q3, Q5 to Q4, Q4 to Q5, R20 to R14, R19 to R15, R19 to R16, R19 to R18, R20 to R19, R19 to R21, R19 to R22, R19 to R23, R19 to R24, R19 to R36, R19 to R49, R2 to R6, R19 to R64, R19 to R68, R19 to R72, R19 to R9, U6 to U4
Other:
- note added: "Low effort measurement (to be confirmed) Imax=2A dRload@2A = 100mV target amp = 30 amp = 1+ (Rf / Rg) = 1 + 10k/0.33k = 31.3"
- note removed: "YOLO measurement Imax=2A dRload@2A = 100mV target amp = 30 amp = 1+ (Rf / Rg) = 1 + 10k/0.33k = 31.3"
