File: outduino.kicad_sch (KiCad schematic)
At the start: 43 parts, among them J3 QWIIC, J3 USB_HDR, J4 USB_C_Receptacle_USB2.0, J5 Lichtenprog_conn, J6 I2C_HDR, Q10 MMBT2222A, Q9 MMBT2222A, SW1 B2, SW1 RST, SW2 B1/BOOT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

Commit message: before scripts
Parts:
- removed J6: I2C_HDR, Connector_PinHeader_2.54mm:PinHeader_1x04_P2.54mm_Vertical, symbol Connector_Generic:Conn_01x04
- removed JP4: 3V3_FROM_USBC, Jumper:SolderJumper-2_P1.3mm_Open_TrianglePad1.0x1.5mm, symbol Jumper:SolderJumper_2_Open
- removed JP5: PWR_FROM_USBC, Jumper:SolderJumper-2_P1.3mm_Open_TrianglePad1.0x1.5mm, symbol Jumper:SolderJumper_2_Open
- removed R16 (x4): 22R/0603, Resistor_SMD:R_0402_1005Metric, symbol Device:R_Small
- added C11 (x2): 10u, Capacitor_SMD:C_0603_1608Metric, symbol Device:C_Small
- added H1 (x2): SCR, MountingHole:MountingHole_3.2mm_M3_Pad_TopOnly, symbol Mechanical:MountingHole_Pad
- added J10: CC1101_CONN, Critbit_lib:8pin_skewed, symbol Connector_Generic:Conn_01x08
- added J3: Conn_01x02, TerminalBlock:TerminalBlock_bornier-2_P5.08mm, symbol Connector_Generic:Conn_01x02
- added TP12 (x5): IOPAD, TestPoint:TestPoint_Pad_D1.0mm, symbol Connector:TestPoint
- added TP12: IOPAD, TestPoint:TestPoint_Pad_D1.5mm, symbol Connector:TestPoint
- C269, C270, C6: footprint Capacitor_SMD:C_0201_0603Metric -> Capacitor_SMD:C_0402_1005Metric
- J3: value USB_HDR -> QWIIC; footprint Connector_PinHeader_2.54mm:PinHeader_1x04_P2.54mm_Vertical -> Connector_JST:JST_SH_SM04B-SRSS-TB_1x04-1MP_P1.00mm_Horizontal
- JP3, JP4, JP5, JP6: footprint Jumper:SolderJumper-3_P1.3mm_Open_RoundedPad1.0x1.5mm -> Jumper:SolderJumper-3_P2.0mm_Open_TrianglePad1.0x1.5mm
- R13: value 33k -> 10k
- R8: footprint Resistor_SMD:R_0201_0603Metric -> Resistor_SMD:R_0402_1005Metric
Connections:
- net PROG_RX is gone; now on net TARG_TX: U3.37 (U0TXD/GPIO43/CLK_OUT1)
- net PROG_TX is gone; now on net TARG_RX: U3.36 (U0RXD/GPIO44/CLK_OUT2)
- net VDD is gone; now on net +3.3V: R2.2
- net +12V: now also J3.2 (Pin_2)
- net +3.3V: now also J3.2 (Pin_2), J5.1 (VDD), C11.1, C11.1, J10.1 (Pin_1), TP12.1
- net ESP_B2: now also U3.17 (GPIO9/TOUCH9/ADC1_CH8/FSPIHD/SUBSPIHD); no longer U3.32 (MTCK/GPIO39/CLK_OUT3/SUBSPICS1)
- net ESP_B3: now also U3.18 (GPIO10/TOUCH10/ADC1_CH9/FSPICS0/FSPIIO4/SUBSPICS0); no longer U3.33 (MTDO/GPIO40/CLK_OUT2)
- net GND: now also J3.1 (Pin_1), C11.2, C11.2, H1.1, H1.1, J10.2 (Pin_2), J3.1 (Pin_1); no longer J3.4 (Pin_4)
- net IN1: now also U3.19 (GPIO11/TOUCH11/ADC2_CH0/FSPID/FSPIIO5/SUBSPID); no longer U3.17 (GPIO9/TOUCH9/ADC1_CH8/FSPIHD/SUBSPIHD)
- net IN2: now also U3.21 (GPIO13/TOUCH13/ADC2_CH2/FSPIQ/FSPIIO7/SUBSPIQ); no longer U3.20 (GPIO12/TOUCH12/ADC2_CH1/FSPICLK/FSPIIO6/SUBSPICLK)
- net IN3: now also U3.25 (GPIO48/SPICLK_N/SUBSPICLK_N_DIFF); no longer U3.8 (GPIO15/U0RTS/ADC2_CH4/XTAL_32K_P)
- net IN4: now also U3.35 (MTMS/GPIO42); no longer U3.11 (GPIO18/U1RXD/ADC2_CH7/CLK_OUT3)
- net OUT1: now also U3.20 (GPIO12/TOUCH12/ADC2_CH1/FSPICLK/FSPIIO6/SUBSPICLK); no longer U3.12 (GPIO8/TOUCH8/ADC1_CH7/SUBSPICS1)
- net OUT2: now also U3.23 (GPIO21); no longer U3.19 (GPIO11/TOUCH11/ADC2_CH0/FSPID/FSPIIO5/SUBSPID)
- net OUT3: now also U3.31 (GPIO38/FSPIWP/SUBSPIWP); no longer U3.22 (GPIO14/TOUCH14/ADC2_CH3/FSPIWP/FSPIDQS/SUBSPIWP)
- net OUT4: now also U3.34 (MTDI/GPIO41/CLK_OUT1); no longer U3.10 (GPIO17/U1TXD/ADC2_CH6)
- net PWR1: now also U3.22 (GPIO14/TOUCH14/ADC2_CH3/FSPIWP/FSPIDQS/SUBSPIWP); no longer U3.7 (GPIO7/TOUCH7/ADC1_CH6)
- net PWR2: now also U3.24 (GPIO47/SPICLK_P/SUBSPICLK_P_DIFF); no longer U3.18 (GPIO10/TOUCH10/ADC1_CH9/FSPICS0/FSPIIO4/SUBSPICS0)
- net PWR3: now also U3.32 (MTCK/GPIO39/CLK_OUT3/SUBSPICS1); no longer U3.21 (GPIO13/TOUCH13/ADC2_CH2/FSPIQ/FSPIIO7/SUBSPIQ)
- net PWR4: now also U3.33 (MTDO/GPIO40/CLK_OUT2); no longer U3.9 (GPIO16/U0CTS/ADC2_CH5/XTAL_32K_NH5)
- net SCL: now also J3.4 (Pin_4), U3.7 (GPIO7/TOUCH7/ADC1_CH6); no longer U3.5 (GPIO5/TOUCH5/ADC1_CH4)
- net SDA: now also J3.3 (Pin_3)
- net USBDM: now also J4.A7 (D-), J4.B7 (D-), TP12.1
- net USBDP: now also J4.A6 (D+), J4.B6 (D+), TP12.1
- net VBUS: now also TP12.1; no longer J3.1 (Pin_1)
- net at J5.8 (5V): now also TP12.1
- net CURR3: now reaches U3.38 (GPIO2/TOUCH2/ADC1_CH1)
- net CURR4: now reaches U3.39 (GPIO1/TOUCH1/ADC1_CH0)
- net CURR2: now reaches U3.4 (GPIO4/TOUCH4/ADC1_CH3)
- new net CC1101_CSn: J10.8 (Pin_8), U3.11 (GPIO18/U1RXD/ADC2_CH7/CLK_OUT3)
- new net CC1101_GDO0: J10.7 (Pin_7), U3.12 (GPIO8/TOUCH8/ADC1_CH7/SUBSPICS1)
- new net CC1101_GDO2: J10.6 (Pin_6), TP12.1
- new net CC1101_SCLK: J10.4 (Pin_4), U3.9 (GPIO16/U0CTS/ADC2_CH5/XTAL_32K_NH5)
- new net CC1101_SI: J10.3 (Pin_3), U3.8 (GPIO15/U0RTS/ADC2_CH4/XTAL_32K_P)
- new net CC1101_SO: J10.5 (Pin_5), U3.10 (GPIO17/U1TXD/ADC2_CH6)
- new net CURR1: U3.5 (GPIO5/TOUCH5/ADC1_CH4)
Other:
- sheet IO_block1 ports: added CURR; removed none
- sheet IO_block2 ports: added CURR; removed none
- sheet IO_block3 ports: added CURR; removed none
- sheet IO_block4 ports: added CURR; removed none
- note added: "<- Connect with wire ->"
- moved on the sheet: J3, R18, R19, R2

Commit message: production
Parts:
- C10, C11, C6: LCSC (none) -> C1525
- C3, C4: LCSC (none) -> C96446
- D1: LCSC (none) -> C2286
- Q10: LCSC (none) -> C8512
- Q9: LCSC (none) -> C15127
- R13: LCSC (none) -> C25744
- R16: LCSC C25117 -> C25890
- R17: LCSC C25117 -> C601102
- R18: LCSC (none) -> C25890
- R19, R2, R8: LCSC (none) -> C25117
- R21, R22: LCSC C25117 -> C25744
- SW1, SW5: LCSC (none) -> C318884
- U2: LCSC (none) -> C6186
Changed lines of the file:
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@@
+      (effects (font (size 1.27 1.27)) hide)
+    )
+    (property "LCSC" "C2286" (at 35.1028 174.2694 0)
       (effects (font (size 1.27 1.27)) hide)
     )
@@
       (effects (font (size 1.27 1.27)) hide)
     )
+    (property "LCSC" "C25117" (at 105.0331 64.77 0)
+      (effects (font (size 1.27 1.27)) hide)
+    )
     (pin "1")
     (pin "2")
@@
       (effects (font (size 1.27 1.27)) hide)
     )
+    (property "LCSC" "C25117" (at 287.3969 30.48 0)
+      (effects (font (size 1.27 1.27)) hide)
+    )
     (pin "1")
     (pin "2")
@@
       (effects (font (size 1.27 1.27)) hide)
     )
-    (property "LCSC" "C25117" (at 63.5 124.46 0)
+    (property "LCSC" "C25744" (at 63.5 124.46 0)
       (effects (font (size 1.27 1.27)) hide)
     )
@@
       (effects (font (size 1.27 1.27)) hide)
     )
+    (property "LCSC" "C318884" (at 383.54 90.17 0)
+      (effects (font (size 1.27 1.27)) hide)
+    )
     (pin "1")
     (pin "2")
@@
       (effects (font (size 1.27 1.27)) hide)
     )
-    (property "LCSC" "C25117" (at 46.99 27.94 0)
+    (property "LCSC" "C25890" (at 46.99 27.94 0)
       (effects (font (size 1.27 1.27)) hide)
     )
@@
     )
     (property "Datasheet" "~" (at 38.1 184.15 0)
+      (effects (font (size 1.27 1.27)) hide)
+    )
+    (property "LCSC" "C25744" (at 36.322 182.9816 0)
       (effects (font (size 1.27 1.27)) hide)
     )
@@
       (effects (font (size 1.27 1.27)) hide)
     )
+    (property "LCSC" "C318884" (at 379.73 48.26 0)
+      (effects (font (size 1.27 1.27)) hide)
+    )
     (pin "1")
     (pin "2")
@@
       (effects (font (size 1.27 1.27)) hide)
     )
+    (property "LCSC" "C96446" (at 44.2341 174.3515 0)
+      (effects (font (size 1.27 1.27)) hide)
+    )
     (pin "1")
     (pin "2")
@@
     )
     (property "Datasheet" "~" (at 60.96 175.26 0)
+      (effects (font (size 1.27 1.27)) hide)
+    )
+    (property "LCSC" "C96446" (at 63.2841 174.3515 0)
       (effects (font (size 1.27 1.27)) hide)
     )
@@
       (effects (font (size 1.27 1.27)) hide)
     )
+    (property "LCSC" "C25117" (at 363.982 35.6616 0)
+      (effects (font (size 1.27 1.27)) hide)
+    )
     (pin "1")
     (pin "2")
@@
       (effects (font (size 1.27 1.27)) hide)
     )
+    (property "LCSC" "C1525" (at 273.2659 103.3116 0)
+      (effects (font (size 1.27 1.27)) hide)
+    )
     (pin "1")
     (pin "2")
@@
       (effects (font (size 1.27 1.27)) hide)
     )
+    (property "LCSC" "C25117" (at 312.42 55.88 0)
+      (effects (font (size 1.27 1.27)) hide)
+    )
     (pin "1")
     (pin "2")
@@
       (effects (font (size 1.27 1.27)) hide)
     )
+    (property "LCSC" "C25890" (at 307.34 55.88 0)
+      (effects (font (size 1.27 1.27)) hide)
+    )
     (pin "1")
     (pin "2")
@@
       (effects (font (size 1.27 1.27)) hide)
     )
-    (property "LCSC" "C25117" (at 46.99 30.48 0)
+    (property "LCSC" "C601102" (at 46.99 30.48 0)
       (effects (font (size 1.27 1.27)) hide)
     )
@@
       (effects (font (size 1.27 1.27)) hide)
     )
-    (property "LCSC" "C25117" (at 63.5 138.43 0)
+    (property "LCSC" "C25744" (at 63.5 138.43 0)
       (effects (font (size 1.27 1.27)) hide)
     )
@@
     )
     (property "Datasheet" "~" (at 73.66 138.43 0)
+      (effects (font (size 1.27 1.27)) hide)
+    )
+    (property "LCSC" "C8512" (at 78.5114 137.5953 0)
       (effects (font (size 1.27 1.27)) hide)
     )
@@
       (effects (font (size 1.27 1.27)) hide)
     )
+    (property "LCSC" "C6186" (at 52.07 165.8452 0)
+      (effects (font (size 1.27 1.27)) hide)
+    )
     (pin "1")
     (pin "2")
@@
       (effects (font (size 1.27 1.27)) hide)
     )
+    (property "LCSC" "C15127" (at 78.5114 123.6253 0)
+      (effects (font (size 1.27 1.27)) hide)
+    )
     (pin "1")
     (pin "2")
@@
       (effects (font (size 1.27 1.27)) hide)
     )
+    (property "LCSC" "C1525" (at 364.7059 212.5316 0)
+      (effects (font (size 1.27 1.27)) hide)
+    )
     (pin "1")
     (pin "2")
@@
     )
     (property "Datasheet" "~" (at 109.22 67.31 0)
+      (effects (font (size 1.27 1.27)) hide)
+    )
+    (property "LCSC" "C25117" (at 110.8669 64.77 0)
       (effects (font (size 1.27 1.27)) hide)
     )
@@
       (effects (font (size 1.27 1.27)) hide)
     )
+    (property "LCSC" "C318884" (at 383.54 111.76 0)
+      (effects (font (size 1.27 1.27)) hide)
+    )
     (pin "1")
     (pin "2")
@@
     )
     (property "Datasheet" "~" (at 365.76 48.26 0)
+      (effects (font (size 1.27 1.27)) hide)
+    )
+    (property "LCSC" "C1525" (at 370.84 46.99 0)
       (effects (font (size 1.27 1.27)) hide)
     )
@@
       (effects (font (size 1.27 1.27)) hide)
     )
+    (property "LCSC" "C1525" (at 363.4359 168.0816 0)
+      (effects (font (size 1.27 1.27)) hide)
+    )
     (pin "1")
     (pin "2")
@@
       (effects (font (size 1.27 1.27)) hide)
     )
+    (property "LCSC" "C1525" (at 282.1559 103.3116 0)
+      (effects (font (size 1.27 1.27)) hide)
+    )
