File: outduino.kicad_sch (KiCad schematic)
At the start: 48 parts, among them J10 CC1101_CONN, J3 Conn_01x02, J3 QWIIC, J4 USB_C_Receptacle_USB2.0, J5 Lichtenprog_conn, Q10 MMBT2222A, Q9 MMBT2222A, SW1 B2, SW1 RST, SW2 B1/BOOT, SW5 B2, U2 AZ1117-3.3, U3 ESP32-S3-WROOM-2

Commit message: add license, update readme
Parts:
- U1: value ~ -> (none)
- renumbered C10 to C1, C269 to C11, C270 to C12, C11 to C16, C11 to C17, C11 to C2, C6 to C8, H1 to H3, J4 to J1, J5 to J2, J3 to J4, J3 to J6, Q9 to Q1, Q10 to Q2, R16 to R2, R8 to R25, R2 to R29, R17 to R3, R2 to R30, R2 to R31, R18 to R4, R19 to R5, R21 to R7, R22 to R8, SW2 to SW3, SW1 to SW4, TP12 to TP1, TP12 to TP2, TP12 to TP3, TP12 to TP4, TP12 to TP5, TP12 to TP6
